File: dual source.sch (KiCad schematic (older format))
At the start: 20 parts, among them P1 BATTERY, P2 CHRG, P3 USB_5PIN_SHELL, P4 ENABLE_5V, P5 ENABLE_3.3V, P6 CONN_01X06, SW1 ON/OFF, U1 SPX3819M5-3.3, U2 LTC3426

Commit message: Board design Attempt 1
Parts:
- SW1: footprint (none) -> ESPlant:SS12D00
- U2: footprint (none) -> freetronics_footprints:SOT23-6
Changed lines of the file:
@@
 F 0 "SW1" H 3700 1350 50  0000 C CNN
 F 1 "ON/OFF" H 3750 1050 50  0000 C CNN
-F 2 "" H 3900 1200 60  0001 C CNN
+F 2 "ESPlant:SS12D00" H 3900 1200 60  0001 C CNN
 F 3 "" H 3900 1200 60  0000 C CNN
 	1    3900 1200
@@
 F 0 "U2" H 5250 2500 60  0000 C CNN
 F 1 "LTC3426" H 5250 3900 60  0000 C CNN
-F 2 "" H 4500 3250 60  0001 C CNN
+F 2 "freetronics_footprints:SOT23-6" H 4500 3250 60  0001 C CNN
 F 3 "" H 4500 3250 60  0000 C CNN
 	1    5250 3200
