File: dual source.kicad_pcb (KiCad board)
At the start: 2 copper layers, 50 x 25 mm, 39 parts, among them P1 BATTERY, P2 CHRG, P3 USB_5PIN_SHELL, P4 EN_5V, P5 EN_3.3V, P6 CONN_01X06, Q201 FDN340P, Q202 FDN340P, Q203 FDN340P, SW1 ON/OFF, U1 SPX3819M5-3.3, U2 LTC3426, U201 CN3063, U202 MCP6002

Commit message: Added photo
Routing:
- net GND: vias 8 -> 1
- net (no net): vias 0 -> 7
Other:
- board text added: "Dual Source battery management by John Spencer http://github.com/mage0r/Dual-Source-Charger TAPR Open Hardware License"
Changed lines of the file:
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@@
-(kicad_pcb (version 4) (host pcbnew 4.0.2-stable)
+(kicad_pcb (version 4) (host pcbnew 4.0.0-rc1-stable)
   (general
     (links 88)
-    (no_connects 1)
-    (area 49.924999 49.924999 100.075001 75.075001)
+    (no_connects 8)
+    (area 48.274629 49.78506 100.156201 75.233509)
     (thickness 1.6)
-    (drawings 4)
+    (drawings 5)
     (tracks 268)
     (zones 0)
@@
     (34 B.Paste user)
     (35 F.Paste user)
-    (36 B.SilkS user)
+    (36 B.SilkS user hide)
     (37 F.SilkS user)
     (38 B.Mask user)
@@
     (visible_elements 7FFFF7FF)
     (pcbplotparams
-      (layerselection 0x00030_80000001)
-      (usegerberextensions false)
+      (layerselection 0x31cff_80000001)
+      (usegerberextensions true)
       (excludeedgelayer true)
       (linewidth 0.500000)
@@
       (outputformat 1)
       (mirror false)
-      (drillshape 1)
+      (drillshape 0)
       (scaleselection 1)
-      (outputdirectory ""))
+      (outputdirectory Gerber/))
   )
   (net 0 "")
@@
       (effects (font (size 0.6 0.6) (thickness 0.1)))
     )
-    (fp_text value SS14 (at 1 2.05) (layer Eco1.User) hide
+    (fp_text value SS14 (at 3.4874 -0.0051 90) (layer Eco1.User) hide
       (effects (font (size 0.5 0.5) (thickness 0.1)))
     )
@@
       (effects (font (size 1 1) (thickness 0.15)))
     )
-    (fp_text value BATTERY (at 2.49682 1.33858 90) (layer F.Fab)
+    (fp_text value BATTERY (at 2.49682 1.33858 90) (layer F.SilkS)
       (effects (font (size 1 1) (thickness 0.15)))
     )
@@
       (effects (font (size 1 1) (thickness 0.15)))
     )
-    (fp_text value CHRG (at -2.34696 1.28778 360) (layer F.Fab)
+    (fp_text value CHRG (at -2.34696 1.28778 360) (layer F.SilkS)
       (effects (font (size 1 1) (thickness 0.15)))
     )
@@
       (effects (font (size 1 1) (thickness 0.15)))
     )
-    (fp_text value EN_5V (at 2.45872 1.17348 180) (layer F.Fab)
+    (fp_text value EN_5V (at 2.45872 1.17348 180) (layer F.SilkS)
       (effects (font (size 1 1) (thickness 0.15)))
     )
@@
       (effects (font (size 1 1) (thickness 0.15)))
     )
-    (fp_text value 1M (at 5.11302 -0.01524) (layer F.Fab)
+    (fp_text value 1M (at 5.11302 -0.01524) (layer F.SilkS)
       (effects (font (size 1 1) (thickness 0.15)))
     )
@@
       (effects (font (size 0.8 0.8) (thickness 0.12)))
     )
-    (fp_text value ON/OFF (at -0.00254 2.58064 90) (layer F.Fab)
+    (fp_text value ON/OFF (at -0.00254 2.58064 90) (layer F.SilkS)
       (effects (font (size 1 1) (thickness 0.15)))
     )
@@
       (net 1 "Net-(C1-Pad1)"))
   )
+  (gr_text "Dual Source battery management\nby John Spencer\n\nhttp://github.com/mage0r/Dual-Source-Charger\nTAPR Open Hardware License" (at 74.0918 59.9694) (layer B.SilkS)
+    (effects (font (size 1 1) (thickness 0.25)) (justify mirror))
+  )
   (gr_line (start 50 75) (end 50 50) (angle 90) (layer Edge.Cuts) (width 0.15))
   (gr_line (start 100 75) (end 50 75) (angle 90) (layer Edge.Cuts) (width 0.15))
@@
   (segment (start 97.55124 52.29606) (end 96.13392 52.29606) (width 0.25) (layer B.Cu) (net 0))
   (segment (start 96.13392 52.29606) (end 96.11868 52.28082) (width 0.25) (layer B.Cu) (net 0))
+  (via (at 63.26886 70.59168) (size 0.6) (drill 0.4) (layers F.Cu B.Cu) (net 0))
+  (via (at 63.16218 53.01996) (size 0.6) (drill 0.4) (layers F.Cu B.Cu) (net 0))
+  (via (at 68.22948 57.531) (size 0.6) (drill 0.4) (layers F.Cu B.Cu) (net 0))
+  (via (at 68.94576 53.19776) (size 0.6) (drill 0.4) (layers F.Cu B.Cu) (net 0))
+  (via (at 75.72756 58.41492) (size 0.6) (drill 0.4) (layers F.Cu B.Cu) (net 0))
+  (via (at 79.31404 57.00268) (size 0.6) (drill 0.4) (layers F.Cu B.Cu) (net 0))
+  (via (at 89.70264 65.532) (size 0.6) (drill 0.4) (layers F.Cu B.Cu) (net 0))
   (segment (start 78.9288 69.6824) (end 80.76688 69.6824) (width 0.25) (layer F.Cu) (net 1))
   (segment (start 90.518 59.7408) (end 91.84384 61.06664) (width 0.25) (layer F.Cu) (net 1))
@@
   (segment (start 75.3466 69.4741) (end 76.2762 69.4741) (width 0.25) (layer F.Cu) (net 1))
   (segment (start 76.4845 69.6824) (end 76.4845 73.0707) (width 0.25) (layer F.Cu) (net 1))
-  (segment (start 84.5515 62.66942) (end 84.5515 60.15738) (width 0.25) (layer F.Cu) (net 2) (status 400000))
+  (segment (start 84.5515 62.66942) (end 84.5515 60.15738) (width 0.25) (layer F.Cu) (net 2))
   (via (at 84.56422 60.14466) (size 0.6) (drill 0.4) (layers F.Cu B.Cu) (net 2))
   (segment (start 84.5515 60.15738) (end 84.56422 60.14466) (width 0.25) (layer F.Cu) (net 2))
-  (via (at 63.26886 70.59168) (size 0.6) (drill 0.4) (layers F.Cu B.Cu) (net 2))
-  (via (at 63.16218 53.01996) (size 0.6) (drill 0.4) (layers F.Cu B.Cu) (net 2))
-  (via (at 68.22948 57.531) (size 0.6) (drill 0.4) (layers F.Cu B.Cu) (net 2))
-  (via (at 68.94576 53.19776) (size 0.6) (drill 0.4) (layers F.Cu B.Cu) (net 2))
-  (via (at 75.72756 58.41492) (size 0.6) (drill 0.4) (layers F.Cu B.Cu) (net 2))
-  (via (at 79.31404 57.00268) (size 0.6) (drill 0.4) (layers F.Cu B.Cu) (net 2))
-  (via (at 89.70264 65.532) (size 0.6) (drill 0.4) (layers F.Cu B.Cu) (net 2))
   (segment (start 54.0766 56.09588) (end 54.0766 57.1449) (width 0.25) (layer F.Cu) (net 2))
   (segment (start 71.54924 64.9605) (end 69.26836 64.9605) (width 0.25) (layer F.Cu) (net 2))
